File: hw/sch_pcb/TFI2CADT01A.kicad_pcb (KiCad board)
At the start: 2 copper layers, 25 x 15 mm, 25 parts, among them J1 SM04B-GHS-TB, J2 SM04B-GHS-TB, J3 SM04B-GHS-TB, J4 SM04B-GHS-TB, M1 HOLE, M2 HOLE, M3 HOLE, M4 HOLE, M5 HOLE, M6 HOLE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

Commit message: Edit PCB
Parts:
- removed D3: LED RED, Mlab_D:LED_1206
- removed R4: 180R, Mlab_R:SMD-0603
- added J5: SM04B-GHS-TB, Connector_JST:JST_GH_SM04B-GHS-TB_1x04-1MP_P1.25mm_Horizontal, B.Cu at (22.2, -16.5)
- added J6: SM04B-GHS-TB, Connector_JST:JST_GH_SM04B-GHS-TB_1x04-1MP_P1.25mm_Horizontal, F.Cu at (22.2, -16.5)
- added JP1: SolderJumper_2_Open, Jumper:SolderJumper-2_P1.3mm_Open_RoundedPad1.0x1.5mm, F.Cu at (14.5, -19.2)
- added JP2: SolderJumper_2_Open, Jumper:SolderJumper-2_P1.3mm_Open_RoundedPad1.0x1.5mm, F.Cu at (10.5, -19.2)
- added R10: 1M, Resistor_SMD:R_0603_1608Metric, B.Cu at (17.0, -16.6)
- added R12: 1M, Resistor_SMD:R_0603_1608Metric, B.Cu at (10.8, -17.9)
- added R13: 887k, Resistor_SMD:R_0603_1608Metric, B.Cu at (8.00, -16.5)
- added R14: 887k, Resistor_SMD:R_0603_1608Metric, B.Cu at (10.8, -20.3)
- added R15: 1M, Resistor_SMD:R_0603_1608Metric, B.Cu at (8.00, -19.7)
- added R16: 10k, Resistor_SMD:R_0603_1608Metric, B.Cu at (16.1, -9.71)
- added R17: 10k, Resistor_SMD:R_0603_1608Metric, B.Cu at (17.9, -9.71)
- added R7: -, Resistor_SMD:R_0603_1608Metric, B.Cu at (14.2, -20.3)
- added R8: 180R, Resistor_SMD:R_0603_1608Metric, B.Cu at (17.0, -19.7)
- added R9: 887k, Resistor_SMD:R_0603_1608Metric, B.Cu at (14.2, -17.9)
- C1: footprint Mlab_R:SMD-0805 -> Capacitor_SMD:C_0805_2012Metric
- C2, C3, C4: footprint Mlab_R:SMD-0603 -> Capacitor_SMD:C_0603_1608Metric
- D1: footprint Mlab_D:LED_1206 -> LED_SMD:LED_0603_1608Metric
- J2: moved to B.Cu
- R1, R2, R3, R5, R6: footprint Mlab_R:SMD-0603 -> Resistor_SMD:R_0603_1608Metric
- U2: value TCA4307 -> LTC4317; footprint Package_SO:VSSOP-8_3.0x3.0mm_P0.65mm -> Package_DFN_QFN:DFN-16-1EP_3x5mm_P0.5mm_EP1.66x4.4mm
- moved R2 11.0 mm to (8.64, -11.2), turned to -90 degrees
- moved J2 9.00 mm to (2.80, -16.5), turned to 90 degrees
- moved M2 8.00 mm to (12.5, -23.0)
- moved M4 8.00 mm to (2.50, -23.0)
- moved M5 8.00 mm to (22.5, -23.0)
- moved C3 7.55 mm to (16.2, -3.76), turned to 0 degrees
- moved R3 7.43 mm to (7.91, -13.8), turned to 180 degrees
- moved R1 6.35 mm to (9.80, -7.06), turned to 90 degrees
- moved C1 6.34 mm to (9.25, -3.51), turned to -90 degrees
- moved R6 6.22 mm to (16.1, -6.44)
- moved D2 6.19 mm to (7.11, -3.91), turned to -90 degrees
- moved C2 6.03 mm to (16.2, -2.03), turned to 0 degrees
- moved D1 6.02 mm to (8.00, -7.00), turned to -90 degrees
- moved U2 5.80 mm to (12.5, -12.9), turned to -90 degrees
- moved U1 4.33 mm to (12.5, -4.42)
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Connections:
- J3 pad 2: /SCLout -> /SCLout1
- J3 pad 3: /SDAout -> /SDAout1
- J4 pad 2: /SCLout -> /SCLout1
- J4 pad 3: /SDAout -> /SDAout1
- R5 pad 2: /SCLout -> /SCLout1
- R6 pad 2: /SDAout -> /SDAout1
- U2 pad 1: +3V3 -> GND
- U2 pad 2: /SCLout -> +3V3
- U2 pad 3: /SCLin -> /XORH2
- U2 pad 4: GND -> /XORL2
- U2 pad 5: Net-(D3-Pad2) -> /XORH1
- U2 pad 6: /SDAin -> /XORL1
- U2 pad 7: /SDAout -> +3V3
Routing:
- net GND: track 23.4 -> 0.00 mm, vias 35 -> 0
- net /SCLout1: track 0.00 -> 20.5 mm, vias 0 -> 3
- net /SCLout2: track 0.00 -> 19.9 mm, vias 0 -> 3
- net /SDAout2: track 0.00 -> 19.7 mm, vias 0 -> 1
- net /SDAout1: track 0.00 -> 17.7 mm, vias 0 -> 1
- net +3V3: track 33.5 -> 49.8 mm, vias 2 -> 8
- net /SDAout: track 14.3 -> 0.00 mm, vias 2 -> 0
- net /SCLout: track 12.8 -> 0.00 mm, vias 2 -> 0
- net /XORL2: track 0.00 -> 10.4 mm, vias 0 -> 1
- net Net-(D3-Pad2): track 9.49 -> 0.00 mm
- net /XORH1: track 0.00 -> 9.39 mm
- net /XORL1: track 0.00 -> 8.91 mm, vias 0 -> 1
- net /XORH2: track 0.00 -> 7.61 mm
- net +5V: track 48.5 -> 55.0 mm, vias 4 -> 5
- net /SDAin: track 18.8 -> 22.8 mm, vias 2 -> 3
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Other:
- board size 25 x 15 mm -> 25 x 23 mm

Commit message: uprava popisu
Parts:
- moved JP1 12.7 mm to (14.8, -6.49), turned to -90 degrees
- moved JP2 5.12 mm to (14.8, -16.5), turned to 90 degrees
- moved C3 0.07 mm to (16.2, -3.69)
Routing:
- net /XORL1: track 8.91 -> 18.0 mm, vias 1 -> 2
- net +5V: track 55.0 -> 64.1 mm, vias 5 -> 3
- net /SCLout1: track 20.5 -> 27.7 mm, vias 3 -> 2
- net +3V3: track 49.8 -> 55.8 mm, vias 8 -> 5
- net /XORL2: track 10.4 -> 14.8 mm, vias 1 -> 2
- net /SDAout1: track 17.7 -> 18.2 mm
- net GND: track 0.00 -> 0.26 mm, vias 0 -> 8
- net /SDAin: track 22.8 -> 22.9 mm, vias 3 -> 2
Other:
- board text added: "0x08 0x0f"
- board text added: "0x78 0x7f"
- board text added: "I2C input (passtrought)"
- board text added: "OUT1"
- board text added: "OUT2"
- board text added: "TFI2CADT01A"

Commit message: oprava teplotnich profilu
Other:
- board text added: "I2C input (pass-trough)"
- board text removed: "I2C input (passtrought)"
Changed lines of the file:
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@@
     (effects (font (size 1 1) (thickness 0.15)))
   )
-  (gr_text "I2C input\n(passtrought)" (at 2.246 -11.494 270) (layer "F.SilkS")
+  (gr_text "I2C input\n(pass-trough)" (at 2.246 -11.494 270) (layer "F.SilkS")
     (effects (font (size 0.8 0.8) (thickness 0.15) bold))
   )
@@
   (segment (start 9.4742 -15.6972) (end 10.448997 -16.671997) (width 0.2) (layer "B.Cu") (net 14))
   (segment (start 10.94221 -16.178784) (end 10.448997 -16.671997) (width 0.2) (layer "B.Cu") (net 14))
+  (zone (net 1) (net_name "GND") (layers F&B.Cu) (hatch edge 0.508)
+    (priority 1)
+    (connect_pads thru_hole_only (clearance 0.2))
+    (min_thickness 0.15) (filled_areas_thickness no)
+    (fill yes (thermal_gap 0.4) (thermal_bridge_width 0.5))
+    (polygon
+      (pts
+        (xy 5.9 -24.560705)
+        (xy 5.9 2.239295)
+        (xy -10.580444 2.28167)
+        (xy -10.9 -24.460705)
+      )
+    )
+  )
   (zone (net 1) (net_name "GND") (layer "F.Cu") (hatch edge 0.508)
     (connect_pads (clearance 0.2))
@@
       )
     )
+  )
+  (zone (net 1) (net_name "GND") (layers F&B.Cu) (hatch edge 0.508)
+    (priority 1)
+    (connect_pads thru_hole_only (clearance 0.2))
+    (min_thickness 0.15) (filled_areas_thickness no)
+    (fill yes (thermal_gap 0.4) (thermal_bridge_width 0.5))
+    (polygon
+      (pts
+        (xy 35.6 -25)
+        (xy 35.6 1.8)
+        (xy 19.119556 1.842375)
+        (xy 18.8 -24.9)
+      )
+    )

Commit message: uprava routingu
Routing:
- net GND: track 0.26 -> 4.22 mm
- net /XORL1: track 18.0 -> 19.0 mm
Other:
- board text added: "2022"
- board text added: "thunderfly.cz"
- board text removed: "PWR"
- board text removed: "READY"
- board text removed: "TFI2CEXT01A"

Commit message: Edit PCB
Parts:
- added G1: LOGO, MLAB_LOGA:TF 10x4,7, F.Cu at (9.50, -11.5)
- moved U1 0.15 mm to (12.5, -4.57)
Routing:
- net /SCLout1: track 27.7 -> 15.8 mm, vias 2 -> 3
- net +5V: track 64.1 -> 57.9 mm
- net /SDAout2: track 20.2 -> 18.2 mm
- net /XORL2: track 14.8 -> 13.2 mm, vias 2 -> 1
- net /SCLout2: track 19.9 -> 18.5 mm
- net /XORL1: track 19.0 -> 17.7 mm, vias 2 -> 1
- net /SDAout1: track 18.2 -> 17.4 mm
- net +3V3: track 55.8 -> 56.5 mm
- net GND: track 4.22 -> 3.96 mm, vias 8 -> 26

Commit message: Edit pcb
Changed lines of the file:
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@@
       (effects (font (size 1 1) (thickness 0.15)) (justify mirror))
     )
-    (fp_text value "-" (at 0 -1.43) (layer "B.Fab")
+    (fp_text value "-" (at 0 -1.43) (layer "B.Fab") hide
       (effects (font (size 1 1) (thickness 0.15)) (justify mirror))
     )
@@
       (effects (font (size 1 1) (thickness 0.15)) (justify mirror))
     )
-    (fp_text value "LED GREEN" (at 0 -1.43 90) (layer "B.Fab")
+    (fp_text value "LED GREEN" (at 0 -1.43 90) (layer "B.Fab") hide
       (effects (font (size 1 1) (thickness 0.15)) (justify mirror))
     )
@@
       (effects (font (size 1 1) (thickness 0.15)) (justify mirror))
     )
-    (fp_text value "100nF" (at 0 -1.43) (layer "B.Fab")
+    (fp_text value "100nF" (at 0 -1.43) (layer "B.Fab") hide
       (effects (font (size 1 1) (thickness 0.15)) (justify mirror))
     )
@@
       (effects (font (size 1 1) (thickness 0.15)) (justify mirror))
     )
-    (fp_text user "${REFERENCE}" (at 0 -1.27 90) (layer "B.Fab")
+    (fp_text user "${REFERENCE}" (at 0.1016 1.27 90) (layer "B.Fab")
       (effects (font (size 1 1) (thickness 0.15)) (justify mirror))
     )
@@
       (effects (font (size 1 1) (thickness 0.15)) (justify mirror))
     )
-    (fp_text value "10k" (at 0 -1.43 90) (layer "B.Fab")
+    (fp_text value "10k" (at 0 -1.43 90) (layer "B.Fab") hide
       (effects (font (size 1 1) (thickness 0.15)) (justify mirror))
     )
@@
       (effects (font (size 1 1) (thickness 0.15)) (justify mirror))
     )
-    (fp_text value "10k" (at 0 -1.43 90) (layer "B.Fab")
+    (fp_text value "10k" (at 0 -1.43 90) (layer "B.Fab") hide
       (effects (font (size 1 1) (thickness 0.15)) (justify mirror))
     )
@@
       (effects (font (size 1 1) (thickness 0.15)) (justify mirror))
     )
-    (fp_text value "1uF" (at 0 -1.43) (layer "B.Fab")
+    (fp_text value "1uF" (at 0 -1.43) (layer "B.Fab") hide
       (effects (font (size 1 1) (thickness 0.15)) (justify mirror))
     )
@@
       (effects (font (size 1 1) (thickness 0.15)) (justify mirror))
     )
-    (fp_text value "1M" (at 0 -1.43 90) (layer "B.Fab")
-      (effects (font (size 1 1) (thickness 0.15)) (justify mirror))
-    )
-    (fp_text user "${REFERENCE}" (at 0 0 90) (layer "B.Fab") hide
+    (fp_text value "1M" (at 0 -1.43 90) (layer "B.Fab") hide
+      (effects (font (size 1 1) (thickness 0.15)) (justify mirror))
+    )
+    (fp_text user "${REFERENCE}" (at 0 0 90) (layer "B.Fab")
       (effects (font (size 0.4 0.4) (thickness 0.06)) (justify mirror))
     )
@@
       (effects (font (size 1 1) (thickness 0.15)) (justify mirror))
     )
-    (fp_text value "1M" (at 0 -1.43) (layer "B.Fab")
+    (fp_text value "1M" (at 0 -1.43) (layer "B.Fab") hide
       (effects (font (size 1 1) (thickness 0.15)) (justify mirror))
     )
@@
       (effects (font (size 1 1) (thickness 0.15)) (justify mirror))
     )
-    (fp_text value "SM04B-GHS-TB" (at 0 -3.9 90) (layer "B.Fab")
+    (fp_text value "SM04B-GHS-TB" (at 0 -3.9 90) (layer "B.Fab") hide
       (effects (font (size 1 1) (thickness 0.15)) (justify mirror))
     )
@@
       (effects (font (size 1 1) (thickness 0.15)) (justify mirror))
     )
-    (fp_text value "180R" (at 0 -1.43 90) (layer "B.Fab")
+    (fp_text value "180R" (at 0 -1.43 90) (layer "B.Fab") hide
       (effects (font (size 1 1) (thickness 0.15)) (justify mirror))
     )
@@
       (effects (font (size 1 1) (thickness 0.15)) (justify mirror))
     )
-    (fp_text value "887k" (at 0 -1.43) (layer "B.Fab")
+    (fp_text value "887k" (at 0 -1.43) (layer "B.Fab") hide
       (effects (font (size 1 1) (thickness 0.15)) (justify mirror))
     )
@@
       (effects (font (size 1 1) (thickness 0.15)) (justify mirror))
     )
-    (fp_text value "887k" (at 0 -1.43 90) (layer "B.Fab")
+    (fp_text value "887k" (at 0 -1.43 90) (layer "B.Fab") hide
       (effects (font (size 1 1) (thickness 0.15)) (justify mirror))
     )
@@
       (effects (font (size 1 1) (thickness 0.15)) (justify mirror))
     )
-    (fp_text value "180R" (at 0 -1.43 90) (layer "B.Fab")
+    (fp_text value "180R" (at 0 -1.43 90) (layer "B.Fab") hide
       (effects (font (size 1 1) (thickness 0.15)) (justify mirror))
     )
@@
       (effects (font (size 1 1) (thickness 0.15)) (justify mirror))
     )
-    (fp_text value "10k" (at 0 -1.43 90) (layer "B.Fab")
+    (fp_text value "10k" (at 0 -1.43 90) (layer "B.Fab") hide
       (effects (font (size 1 1) (thickness 0.15)) (justify mirror))
     )
@@
       (effects (font (size 1 1) (thickness 0.15)) (justify mirror))
     )
-    (fp_text value "10k" (at 0 -1.43 90) (layer "B.Fab")
+    (fp_text value "10k" (at 0 -1.43 90) (layer "B.Fab") hide
       (effects (font (size 1 1) (thickness 0.15)) (justify mirror))
     )
@@
       (effects (font (size 1 1) (thickness 0.15)) (justify mirror))
     )
-    (fp_text value "887k" (at 0 -1.43) (layer "B.Fab")
+    (fp_text value "887k" (at 0 -1.43) (layer "B.Fab") hide
       (effects (font (size 1 1) (thickness 0.15)) (justify mirror))
     )
@@
       (effects (font (size 1 1) (thickness 0.15)) (justify mirror))
     )
-    (fp_text value "10k" (at 0 -1.43) (layer "B.Fab")
+    (fp_text value "10k" (at 0 -1.43) (layer "B.Fab") hide
       (effects (font (size 1 1) (thickness 0.15)) (justify mirror))
     )
@@
       (effects (font (size 1 1) (thickness 0.15)) (justify mirror))
     )
-    (fp_text value "10k" (at 0 -1.43 90) (layer "B.Fab")
+    (fp_text value "10k" (at 0 -1.43 90) (layer "B.Fab") hide
       (effects (font (size 1 1) (thickness 0.15)) (justify mirror))
     )
@@
       (effects (font (size 1 1) (thickness 0.15)) (justify mirror))
     )
-    (fp_text value "LTC4317" (at 0 -3.55 90) (layer "B.Fab")
+    (fp_text value "LTC4317" (at 0 -3.55 90) (layer "B.Fab") hide
       (effects (font (size 1 1) (thickness 0.15)) (justify mirror))
     )
@@
       (effects (font (size 1 1) (thickness 0.15)) (justify mirror))
     )
-    (fp_text value "10uF" (at 0 -1.68 90) (layer "B.Fab")
+    (fp_text value "10uF" (at 0 -1.68 90) (layer "B.Fab") hide
       (effects (font (size 1 1) (thickness 0.15)) (justify mirror))
     )
@@
       (effects (font (size 1 1) (thickness 0.15)) (justify mirror))
     )
-    (fp_text value "1M" (at 0 -1.43 90) (layer "B.Fab")
+    (fp_text value "1M" (at 0 -1.43 90) (layer "B.Fab") hide
       (effects (font (size 1 1) (thickness 0.15)) (justify mirror))
     )
@@
       (effects (font (size 1 1) (thickness 0.15)) (justify mirror))
     )
-    (fp_text value "100nF" (at 0 -1.43 90) (layer "B.Fab")
+    (fp_text value "100nF" (at 0 -1.43 90) (layer "B.Fab") hide
       (effects (font (size 1 1) (thickness 0.15)) (justify mirror))
     )
@@
   (zone (net 1) (net_name "GND") (layers F&B.Cu) (hatch edge 0.508)
     (priority 1)
-    (connect_pads thru_hole_only (clearance 0.2))
+    (connect_pads yes (clearance 0.2))
     (min_thickness 0.15) (filled_areas_thickness no)
     (fill yes (thermal_gap 0.4) (thermal_bridge_width 0.5))
@@
     )
   )
-  (zone (net 1) (net_name "GND") (layers F&B.Cu) (hatch edge 0.508)
+  (zone (net 1) (net_name "GND") (layer "B.Cu") (hatch edge 0.508)
     (priority 1)
-    (connect_pads thru_hole_only (clearance 0.2))
+    (connect_pads yes (clearance 0.2))
     (min_thickness 0.15) (filled_areas_thickness no)
     (fill yes (thermal_gap 0.4) (thermal_bridge_width 0.5))
     (polygon
       (pts
-        (xy 35.6 -25)
-        (xy 35.6 1.8)
-        (xy 19.119556 1.842375)
-        (xy 18.8 -24.9)
+        (xy 44.45 1.27)
+        (xy 19.05 1.27)
+        (xy 19.05 -27.94)
+        (xy 44.45 -27.94)
       )
     )
