File: hw/sch_pcb/TFI2CADT01.kicad_pcb (KiCad board)
At the start: 2 copper layers, 25 x 23 mm, 38 parts, among them J1 SM04B-GHS-TB, J2 SM04B-GHS-TB, J3 SM04B-GHS-TB, J4 SM04B-GHS-TB, J5 SM04B-GHS-TB, J6 SM04B-GHS-TB, M1 HOLE, M2 HOLE, M3 HOLE, M4 HOLE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

Commit message: Upravy pred vyrobou
Parts:
- moved G1 0.50 mm to (137.3, 104.1)
- moved J1 0.50 mm to (131.6, 109.1)
- moved J2 0.50 mm to (131.6, 99.1)
- moved J3 0.50 mm to (150.0, 109.1)
- moved J4 0.50 mm to (150.0, 109.1)
- moved J5 0.50 mm to (150.0, 99.1)
- moved J6 0.50 mm to (150.0, 99.1)
- moved JP1 0.50 mm to (142.6, 109.1)
- moved JP2 0.50 mm to (142.6, 99.1)
- moved D2 0.26 mm to (135.6, 111.6)
- moved R13 0.25 mm to (136.5, 99.0)
- moved R15 0.25 mm to (136.5, 95.8)
- moved R10 0.24 mm to (145.0, 99.0)
- moved R8 0.24 mm to (145.0, 95.9)
- moved R17 0.13 mm to (146.1, 105.9)
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Routing:
- net +5V: track 57.9 -> 61.4 mm
- net /XORL2: track 13.2 -> 12.4 mm
- net /SCLin: track 19.7 -> 20.5 mm
Other:
- board text added: "2023"
- board text added: "TFI2CADT01B"
- board text removed: "2022"
- board text removed: "TFI2CADT01A"
