File: hw/sch_pcb/TFI2CADT01.kicad_sch (KiCad schematic)
At the start: 38 parts, among them J1 SM04B-GHS-TB, J2 SM04B-GHS-TB, J3 SM04B-GHS-TB, J4 SM04B-GHS-TB, J5 SM04B-GHS-TB, J6 SM04B-GHS-TB, M1 HOLE, M2 HOLE, M3 HOLE, M4 HOLE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

Commit message: Edit UST_ID
Parts:
- R13, R14, R9: UST_ID 61e02cad2eac0c9aef5c894c -> 6272c899dc56076e9a222bfe
Changed lines of the file:
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@@
       (effects (font (size 1.27 1.27)) hide)
     )
-    (property "UST_ID" "61e02cad2eac0c9aef5c894c" (at 131.445 156.21 0)
+    (property "UST_ID" "6272c899dc56076e9a222bfe" (at 131.445 156.21 0)
       (effects (font (size 1.27 1.27)) hide)
     )
@@
       (effects (font (size 1.27 1.27)) hide)
     )
-    (property "UST_ID" "61e02cad2eac0c9aef5c894c" (at 158.115 156.21 0)
+    (property "UST_ID" "6272c899dc56076e9a222bfe" (at 158.115 156.21 0)
       (effects (font (size 1.27 1.27)) hide)
     )
@@
       (effects (font (size 1.27 1.27)) hide)
     )
-    (property "UST_ID" "61e02cad2eac0c9aef5c894c" (at 156.845 133.35 0)
-      (effects (font (size 1.27 1.27)) hide)
-    )
+    (property "UST_ID" "6272c899dc56076e9a222bfe" (at 156.845 133.35 0)
+      (effects (font (size 1.27 1.27)) hide)
+    )

Commit message: Aktualizace metadat
Parts:
- JP1, JP2, M1, M2, M3, M4, M5, M6: now left out of the parts list
Changed lines of the file:
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@@
   )
   (symbol (lib_id "Jumper:SolderJumper_2_Open") (at 130.81 146.685 0) (unit 1)
-    (in_bom yes) (on_board yes) (dnp no) (fields_autoplaced)
+    (in_bom no) (on_board yes) (dnp no) (fields_autoplaced)
     (property "Reference" "JP1" (at 130.81 143.2306 0)
       (effects (font (size 1.27 1.27)))
@@
   )
   (symbol (lib_id "MLAB_MECHANICAL:HOLE_TF") (at 273.05 21.59 90) (unit 1)
-    (in_bom yes) (on_board yes) (dnp no) (fields_autoplaced)
+    (in_bom no) (on_board yes) (dnp no) (fields_autoplaced)
     (property "Reference" "M6" (at 274.4471 20.2579 90)
       (effects (font (size 1.524 1.524)) (justify right))
@@
   )
   (symbol (lib_id "MLAB_MECHANICAL:HOLE_TF") (at 255.27 21.59 90) (unit 1)
-    (in_bom yes) (on_board yes) (dnp no) (fields_autoplaced)
+    (in_bom no) (on_board yes) (dnp no) (fields_autoplaced)
     (property "Reference" "M4" (at 256.6671 20.2579 90)
       (effects (font (size 1.524 1.524)) (justify right))
@@
   )
   (symbol (lib_id "MLAB_MECHANICAL:HOLE_TF") (at 246.38 21.59 90) (unit 1)
-    (in_bom yes) (on_board yes) (dnp no)
+    (in_bom no) (on_board yes) (dnp no)
     (property "Reference" "M3" (at 247.7771 20.2579 90)
       (effects (font (size 1.524 1.524)) (justify right))
@@
   )
   (symbol (lib_id "Jumper:SolderJumper_2_Open") (at 158.115 146.685 0) (unit 1)
-    (in_bom yes) (on_board yes) (dnp no) (fields_autoplaced)
+    (in_bom no) (on_board yes) (dnp no) (fields_autoplaced)
     (property "Reference" "JP2" (at 158.115 143.2306 0)
       (effects (font (size 1.27 1.27)))
@@
   )
   (symbol (lib_id "MLAB_MECHANICAL:HOLE_TF") (at 237.49 21.59 90) (unit 1)
-    (in_bom yes) (on_board yes) (dnp no) (fields_autoplaced)
+    (in_bom no) (on_board yes) (dnp no) (fields_autoplaced)
     (property "Reference" "M2" (at 238.8871 20.2579 90)
       (effects (font (size 1.524 1.524)) (justify right))
@@
   )
   (symbol (lib_id "MLAB_MECHANICAL:HOLE_TF") (at 228.6 21.59 90) (unit 1)
-    (in_bom yes) (on_board yes) (dnp no) (fields_autoplaced)
+    (in_bom no) (on_board yes) (dnp no) (fields_autoplaced)
     (property "Reference" "M1" (at 229.9971 20.2579 90)
       (effects (font (size 1.524 1.524)) (justify right))
@@
   )
   (symbol (lib_id "MLAB_MECHANICAL:HOLE_TF") (at 264.16 21.59 90) (unit 1)
-    (in_bom yes) (on_board yes) (dnp no) (fields_autoplaced)
+    (in_bom no) (on_board yes) (dnp no) (fields_autoplaced)
     (property "Reference" "M5" (at 265.5571 20.2579 90)
       (effects (font (size 1.524 1.524)) (justify right))
